Commit message: Update fr3v6 configuration to use new joint names and enable loop animation

File: frcobot_description/urdf/fr3v6.urdf (robot description, URDF)
Before this commit: robot fr3v6, 9 links, 8 joints
Links:
- removed link base_link
- removed link j1_Link
- removed link j2_Link
- removed link j3_Link
- removed link j4_Link
- removed link j5_Link
- removed link j6_Link
- removed link tool_Link
- added link fr3_base_link, mass 0.78393; collision mesh filename=package://frcobot_description/meshes/fr3v6/collision/base_l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; visual mesh filename=package://frcobot_description/meshes/fr3v6/visual/base_link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
- added link fr3_j1_Link, mass 2.1225; collision mesh filename=package://frcobot_description/meshes/fr3v6/collision/j1_Lin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; visual mesh filename=package://frcobot_description/meshes/fr3v6/visual/j1_Link.D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
- added link fr3_j2_Link, mass 4.8053; collision mesh filename=package://frcobot_description/meshes/fr3v6/collision/j2_Lin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; visual mesh filename=package://frcobot_description/meshes/fr3v6/visual/j2_Link.D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
- added link fr3_j3_Link, mass 2.2312; collision mesh filename=package://frcobot_description/meshes/fr3v6/collision/j3_Lin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; visual mesh filename=package://frcobot_description/meshes/fr3v6/visual/j3_Link.D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
- added link fr3_j4_Link, mass 1.5961; collision mesh filename=package://frcobot_description/meshes/fr3v6/collision/j4_Lin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; visual mesh filename=package://frcobot_description/meshes/fr3v6/visual/j4_Link.D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
- added link fr3_j5_Link, mass 1.5961; collision mesh filename=package://frcobot_description/meshes/fr3v6/collision/j5_Lin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; visual mesh filename=package://frcobot_description/meshes/fr3v6/visual/j5_Link.D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
- added link fr3_j6_Link, mass 0.53877; collision mesh filename=package://frcobot_description/meshes/fr3v6/collision/j6_Lin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; visual mesh filename=package://frcobot_description/meshes/fr3v6/visual/j6_Link.D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
- added link fr3_tool_Link, mass 0; collision box size=0 0 0; visual box size=0 0 0
Joints:
- removed joint j1
- removed joint j2
- removed joint j3
- removed joint j4
- removed joint j5
- removed joint j6
- removed joint tool
- added joint fr3_j1: type revolute, parent fr3_base_link, child fr3_j1_Link, origin xyz=0 0 0 rpy=0 0 0, axis 0 0 1, limit lower=-3.0543 upper=3.0543 effort=150 velocity=3.15
- added joint fr3_j2: type revolute, parent fr3_j1_Link, child fr3_j2_Link, origin xyz=0 0 0.14 rpy=1.5708 0 0, axis 0 0 1, limit lower=-4.6251 upper=1.4835 effort=150 velocity=3.15
- added joint fr3_j3: type revolute, parent fr3_j2_Link, child fr3_j3_Link, origin xyz=-0.28 0 0 rpy=0 0 0, axis 0 0 1, limit lower=-2.8274 upper=2.8274 effort=150 velocity=3.15
- added joint fr3_j4: type revolute, parent fr3_j3_Link, child fr3_j4_Link, origin xyz=-0.24001 0 0 rpy=0 0 0, axis 0 0 1, limit lower=-4.6251 upper=1.4835 effort=28 velocity=3.2
- added joint fr3_j5: type revolute, parent fr3_j4_Link, child fr3_j5_Link, origin xyz=0 0 0.102 rpy=1.5708 0 0, axis 0 0 1, limit lower=-3.0543 upper=3.0543 effort=28 velocity=3.2
- added joint fr3_j6: type revolute, parent fr3_j5_Link, child fr3_j6_Link, origin xyz=0 0 0.102 rpy=-1.5708 0 0, axis 0 0 1, limit lower=-3.0543 upper=3.0543 effort=28 velocity=3.2
- added joint fr3_tool: type fixed, parent fr3_j6_Link, child fr3_tool_Link, origin xyz=0 0 0.1 rpy=0 0 0, axis 0 0 1, limit lower=0 upper=0 effort=0 velocity=0
- joint world: child base_link -> fr3_base_link
